File: pcb/141-000-switch-matrix.kicad_sch (KiCad schematic)
At the start: 124 parts, among them SW1 SW_Push, SW10 SW_Push, SW11 SW_Push, SW12 SW_Push, SW13 SW_Push, SW14 SW_Push, SW15 SW_Push, SW16 SW_Push, SW17 SW_Push, SW18 SW_Push, SW19 SW_Push, SW2 SW_Push, SW20 SW_Push, SW21 SW_Push, SW22 SW_Push, SW23 SW_Push, SW24 SW_Push, SW25 SW_Push, SW26 SW_Push, SW27 SW_Push, SW28 SW_Push, SW29 SW_Push, SW3 SW_Push, SW30 SW_Push, SW31 SW_Push, SW32 SW_Push, SW33 SW_Push, SW34 SW_Push, SW35 SW_Push, SW36 SW_Push, SW37 SW_Push, SW38 SW_Push, SW39 SW_Push, SW4 SW_Push, SW40 SW_Push, SW41 SW_Push, SW43 SW_Push, SW44 SW_Push, SW45 SW_Push, SW46 SW_Push, SW47 SW_Push, SW48 SW_Push, SW49 SW_Push, SW5 SW_Push, SW50 SW_Push, SW51 SW_Push, SW52 SW_Push, SW53 SW_Push, SW54 SW_Push, SW57 SW_Push, SW58 SW_Push, SW59 SW_Push, SW6 SW_Push, SW60 SW_Push, SW61 SW_Push, SW62 SW_Push, SW63 SW_Push, SW64 SW_Push, SW65 SW_Push, SW7 SW_Push, SW8 SW_Push, SW9 SW_Push

Commit message: add git ignore, and new sheets etc
Parts:
- D10, D11, D12, D13, D14, D15, D16, D17, D18, D19, D20, D21, D22, D23, D24, D25, D26, D27, D28, D29, D30, D31, D32, D33, D34, D35, D36, D37, D38, D39, D4, D40, D41, D42, D43, D44, D46, D47, D48, D49, D5, D50, D51, D52, D53, D54, D55, D56, D57, D6, D60, D61, D62, D63, D64, D65, D66, D67, D68, D7, D8, D9: footprint (none) -> Diode_SMD:D_0402_1005Metric
- SW1, SW10, SW11, SW12, SW13, SW16, SW17, SW18, SW19, SW2, SW20, SW21, SW22, SW23, SW24, SW25, SW26, SW27, SW3, SW30, SW31, SW32, SW33, SW34, SW35, SW36, SW37, SW38, SW39, SW4, SW40, SW44, SW45, SW46, SW47, SW48, SW49, SW5, SW50, SW51, SW52, SW6, SW7, SW8, SW9: footprint Kahil Switches:SW_Kailh_Choc_Mini_1.00u -> Kahil Switches:SW_Kailh_Choc_V2_1.00u
- SW14: footprint Kahil Switches:SW_Kailh_Choc_Mini_2.00u -> Kahil Switches:SW_Kailh_Choc_V2_2.00u
- SW15: footprint Kahil Switches:SW_Kailh_Choc_Mini_1.00u -> Kahil Switches:SW_Kailh_Choc_V2_1.50u
- SW28: footprint Kahil Switches:SW_Kailh_Choc_Mini_1.50u -> Kahil Switches:SW_Kailh_Choc_V2_1.50u
- SW29: footprint Kahil Switches:SW_Kailh_Choc_Mini_1.75u -> Kahil Switches:SW_Kailh_Choc_V2_1.75u
- SW41: footprint Kahil Switches:SW_Kailh_Choc_Mini_2.25u -> Kahil Switches:SW_Kailh_Choc_V2_2.25u
- SW43: footprint Kahil Switches:SW_Kailh_Choc_Mini_1.00u -> Kahil Switches:SW_Kailh_Choc_V2_2.25u
- SW53: footprint Kahil Switches:SW_Kailh_Choc_Mini_2.75u -> Kahil Switches:SW_Kailh_Choc_V2_1.00u
- SW54: footprint Kahil Switches:SW_Kailh_Choc_Mini_1.25u -> Kahil Switches:SW_Kailh_Choc_V2_2.75u
- SW57, SW58, SW62, SW63: footprint Kahil Switches:SW_Kailh_Choc_Mini_1.25u -> Kahil Switches:SW_Kailh_Choc_V2_1.25u
- SW59: footprint Kahil Switches:SW_Kailh_Choc_Mini_3.00u -> Kahil Switches:SW_Kailh_Choc_V2_1.25u
- SW60: footprint Kahil Switches:SW_Kailh_Choc_Mini_3.00u -> Kahil Switches:SW_Kailh_Choc_V2_3.00u
- SW61: footprint Kahil Switches:SW_Kailh_Choc_Mini_1.25u -> Kahil Switches:SW_Kailh_Choc_V2_3.00u
- SW64: footprint Kahil Switches:SW_Kailh_Choc_Mini_1.50u -> Kahil Switches:SW_Kailh_Choc_V2_1.25u
- SW65: footprint (none) -> Kahil Switches:SW_Kailh_Choc_V2_1.50u

Commit message: major keyboard components completed
Connections:
- net COLUMN 10: now also SW51.2, SW61.2; no longer SW52.2
- net COLUMN 11: now also SW52.2, SW62.2; no longer SW53.2
- net COLUMN 12: now also SW53.2, SW63.2; no longer SW54.2
- net COLUMN 13: now also SW64.2; no longer SW41.2
- net COLUMN 14: now also SW41.2, SW54.2, SW65.2
- net COLUMN 5: no longer SW61.2
- net COLUMN 6: no longer SW48.2, SW62.2
- net COLUMN 7: now also SW48.2; no longer SW49.2, SW63.2
- net COLUMN 8: now also SW49.2; no longer SW50.2, SW64.2
- net COLUMN 9: now also SW50.2; no longer SW51.2, SW65.2
Other:
- moved on the sheet: D44, D51, D52, D53, D54, D55, D56, D57, D64, D65, D66, D67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
