File: pcb/writerdeck.kicad_pcb (KiCad board)
At the start: 2 copper layers, 132 parts, among them SW1 SW_Push, SW10 SW_Push, SW11 SW_Push, SW12 SW_Push, SW13 SW_Push, SW14 SW_Push, SW15 SW_Push, SW16 SW_Push, SW17 SW_Push, SW18 SW_Push, SW19 SW_Push, SW2 SW_Push, SW20 SW_Push, SW21 SW_Push, SW22 SW_Push, SW23 SW_Push, SW24 SW_Push, SW25 SW_Push, SW26 SW_Push, SW27 SW_Push, SW28 SW_Push, SW29 SW_Push, SW3 SW_Push, SW30 SW_Push, SW31 SW_Push, SW32 SW_Push, SW33 SW_Push, SW34 SW_Push, SW35 SW_Push, SW36 SW_Push, SW37 SW_Push, SW38 SW_Push, SW39 SW_Push, SW4 SW_Push, SW40 SW_Push, SW41 SW_Push, SW43 SW_Push, SW44 SW_Push, SW45 SW_Push, SW46 SW_Push, SW47 SW_Push, SW48 SW_Push, SW49 SW_Push, SW5 SW_Push, SW50 SW_Push, SW51 SW_Push, SW52 SW_Push, SW53 SW_Push, SW54 SW_Push, SW57 SW_Push, SW58 SW_Push, SW59 SW_Push, SW6 SW_Push, SW60 SW_Push, SW61 SW_Push, SW62 SW_Push, SW63 SW_Push, SW64 SW_Push, SW65 SW_Push, SW7 SW_Push, SW8 SW_Push, SW9 SW_Push, U1 MCP73871, U2 TPS61090, U3 NCP1117-3.3_SOT223, U4 USB6B1, U5 RP2040, U6 W25Q16JVSS, Y1 ABM8-272-T3

Commit message: major keyboard components completed
Parts:
- added C1: 10uF, Capacitor_SMD:C_0402_1005Metric, F.Cu at (143.6, 199.0)
- added C10: 100n, Capacitor_SMD:C_0402_1005Metric, F.Cu at (199.1, 123.2)
- added C11: 100n, Capacitor_SMD:C_0402_1005Metric, F.Cu at (197.1, 123.2)
- added C12: 100n, Capacitor_SMD:C_0402_1005Metric, F.Cu at (197.1, 125.1)
- added C13: 100n, Capacitor_SMD:C_0402_1005Metric, F.Cu at (198.1, 125.1)
- added C14: 100n, Capacitor_SMD:C_0402_1005Metric, F.Cu at (199.1, 125.1)
- added C15: 1u, Capacitor_SMD:C_0402_1005Metric, B.Cu at (200.4, 128.7)
- added C16: 1u, Capacitor_SMD:C_0402_1005Metric, B.Cu at (198.9, 129.2)
- added C17: 100n, Capacitor_SMD:C_0402_1005Metric, F.Cu at (198.1, 118.7)
- added C18: 100n, Capacitor_SMD:C_0402_1005Metric, F.Cu at (199.2, 118.7)
- added C19: 100n, Capacitor_SMD:C_0402_1005Metric, B.Cu at (197.8, 134.3)
- added C2: 0.1uF, Capacitor_SMD:C_0402_1005Metric, F.Cu at (143.6, 201.0)
- added C20: 15p, Capacitor_SMD:C_0402_1005Metric, B.Cu at (192.8, 120.4)
- added C21: 15p, Capacitor_SMD:C_0402_1005Metric, B.Cu at (188.3, 121.2)
- added C3: 10uF, Capacitor_SMD:C_0402_1005Metric, F.Cu at (143.6, 202.9)
- added C4: 2.2uF, Capacitor_SMD:C_0402_1005Metric, F.Cu at (143.6, 204.9)
- added C5: 100uF, Capacitor_SMD:C_0402_1005Metric, F.Cu at (143.6, 206.9)
- added C6: 10u, Capacitor_SMD:C_0402_1005Metric, F.Cu at (207.0, 126.7)
- added C7: 10u, Capacitor_SMD:C_0402_1005Metric, F.Cu at (207.0, 129.1)
- added C8: 100n, Capacitor_SMD:C_0402_1005Metric, F.Cu at (198.1, 123.2)
- added C9: 100n, Capacitor_SMD:C_0402_1005Metric, F.Cu at (196.1, 125.1)
- added R1: 1k, Resistor_SMD:R_0402_1005Metric, F.Cu at (147.0, 218.4)
- added R10: 200k, Resistor_SMD:R_0402_1005Metric, F.Cu at (152.8, 220.4)
- added R11: 1k, Resistor_SMD:R_0402_1005Metric, F.Cu at (152.8, 222.4)
- added R12: 200k, Resistor_SMD:R_0402_1005Metric, F.Cu at (152.8, 224.3)
- added R13: 5k1, Resistor_SMD:R_0402_1005Metric, F.Cu at (147.0, 228.3)
- added R14: 5k1, Resistor_SMD:R_0402_1005Metric, F.Cu at (147.0, 230.3)
- added R15: DNF (10k), Resistor_SMD:R_0402_1005Metric, F.Cu at (192.5, 133.8)
- added R16: 1k, Resistor_SMD:R_0402_1005Metric, F.Cu at (186.7, 133.7)
- added R17: 1k, Resistor_SMD:R_0402_1005Metric, F.Cu at (190.4, 120.2)
- added R18: 27, Resistor_SMD:R_0402_1005Metric, F.Cu at (142.1, 224.3)
- added R19: 27, Resistor_SMD:R_0402_1005Metric, F.Cu at (142.1, 226.3)
- added R2: 100k, Resistor_SMD:R_0402_1005Metric, F.Cu at (147.0, 220.4)
- added R3: 270k, Resistor_SMD:R_0402_1005Metric, F.Cu at (147.0, 222.4)
- added R4: 100k, Resistor_SMD:R_0402_1005Metric, F.Cu at (147.0, 224.3)
- added R5: 1k, Resistor_SMD:R_0402_1005Metric, F.Cu at (149.9, 218.4)
- added R6: 1k, Resistor_SMD:R_0402_1005Metric, F.Cu at (149.9, 220.4)
- added R7: 1.87m, Resistor_SMD:R_0402_1005Metric, F.Cu at (149.9, 222.4)
- added R8: 340k, Resistor_SMD:R_0402_1005Metric, F.Cu at (149.9, 224.3)
- added R9: 1.07m, Resistor_SMD:R_0402_1005Metric, F.Cu at (152.8, 218.4)
- moved TH1 464.4 mm to (95.3, 234.8)
- moved U2 464.4 mm to (97.4, 225.7)
- moved U4 464.4 mm to (101.3, 236.4)
- moved U1 464.4 mm to (96.7, 216.3)
- moved Y1 446.0 mm to (190.6, 121.0)
- moved U3 445.2 mm to (207.3, 129.0)
- moved D14 445.0 mm to (311.6, 44.2)
- moved D15 445.0 mm to (273.6, 44.2)
- moved D20 445.0 mm to (130.1, 62.2)
- moved D33 445.0 mm to (115.8, 80.9)
- moved D41 445.0 mm to (268.1, 81.0)
- moved D7 445.0 mm to (140.1, 44.2)
- moved SW1 445.0 mm to (80.8, 51.8)
- moved SW12 445.0 mm to (290.4, 51.8)
- moved SW14 445.0 mm to (338.0, 51.8)
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Connections:
- SW41 pad 2: /140-000 Keybaord/141-000 Switch Matrix/COLUMN 13 -> /140-000 Keybaord/141-000 Switch Matrix/COLUMN 14
- SW48 pad 2: /140-000 Keybaord/141-000 Switch Matrix/COLUMN 6 -> /140-000 Keybaord/141-000 Switch Matrix/COLUMN 7
- SW49 pad 2: /140-000 Keybaord/141-000 Switch Matrix/COLUMN 7 -> /140-000 Keybaord/141-000 Switch Matrix/COLUMN 8
- SW50 pad 2: /140-000 Keybaord/141-000 Switch Matrix/COLUMN 8 -> /140-000 Keybaord/141-000 Switch Matrix/COLUMN 9
- SW51 pad 2: /140-000 Keybaord/141-000 Switch Matrix/COLUMN 9 -> /140-000 Keybaord/141-000 Switch Matrix/COLUMN 10
- SW52 pad 2: /140-000 Keybaord/141-000 Switch Matrix/COLUMN 10 -> /140-000 Keybaord/141-000 Switch Matrix/COLUMN 11
- SW53 pad 2: /140-000 Keybaord/141-000 Switch Matrix/COLUMN 11 -> /140-000 Keybaord/141-000 Switch Matrix/COLUMN 12
- SW54 pad 2: /140-000 Keybaord/141-000 Switch Matrix/COLUMN 12 -> /140-000 Keybaord/141-000 Switch Matrix/COLUMN 14
- SW61 pad 2: /140-000 Keybaord/141-000 Switch Matrix/COLUMN 5 -> /140-000 Keybaord/141-000 Switch Matrix/COLUMN 10
- SW62 pad 2: /140-000 Keybaord/141-000 Switch Matrix/COLUMN 6 -> /140-000 Keybaord/141-000 Switch Matrix/COLUMN 11
- SW63 pad 2: /140-000 Keybaord/141-000 Switch Matrix/COLUMN 7 -> /140-000 Keybaord/141-000 Switch Matrix/COLUMN 12
- SW64 pad 2: /140-000 Keybaord/141-000 Switch Matrix/COLUMN 8 -> /140-000 Keybaord/141-000 Switch Matrix/COLUMN 13
- SW65 pad 2: /140-000 Keybaord/141-000 Switch Matrix/COLUMN 9 -> /140-000 Keybaord/141-000 Switch Matrix/COLUMN 14
- U5 pad 11: /140-000 Keybaord/141-000 Switch Matrix/COLUMN 9 -> unconnected-(U5-GPIO8-Pad11)
- U5 pad 12: /140-000 Keybaord/141-000 Switch Matrix/COLUMN 10 -> unconnected-(U5-GPIO9-Pad12)
- U5 pad 13: /140-000 Keybaord/141-000 Switch Matrix/COLUMN 11 -> unconnected-(U5-GPIO10-Pad13)
- U5 pad 14: /140-000 Keybaord/141-000 Switch Matrix/COLUMN 12 -> unconnected-(U5-GPIO11-Pad14)
- U5 pad 15: /140-000 Keybaord/141-000 Switch Matrix/COLUMN 13 -> unconnected-(U5-GPIO12-Pad15)
- U5 pad 16: /140-000 Keybaord/141-000 Switch Matrix/COLUMN 14 -> unconnected-(U5-GPIO13-Pad16)
- U5 pad 30: unconnected-(U5-GPIO19-Pad30) -> /140-000 Keybaord/141-000 Switch Matrix/COLUMN 8
- U5 pad 31: unconnected-(U5-GPIO20-Pad31) -> /140-000 Keybaord/141-000 Switch Matrix/COLUMN 9
- U5 pad 32: unconnected-(U5-GPIO21-Pad32) -> /140-000 Keybaord/141-000 Switch Matrix/COLUMN 10
- U5 pad 34: unconnected-(U5-GPIO22-Pad34) -> /140-000 Keybaord/141-000 Switch Matrix/COLUMN 11
- U5 pad 35: unconnected-(U5-GPIO23-Pad35) -> /140-000 Keybaord/141-000 Switch Matrix/COLUMN 12
- U5 pad 36: unconnected-(U5-GPIO24-Pad36) -> /140-000 Keybaord/141-000 Switch Matrix/COLUMN 13
- U5 pad 37: unconnected-(U5-GPIO25-Pad37) -> /140-000 Keybaord/141-000 Switch Matrix/COLUMN 14
- U5 pad 9: /140-000 Keybaord/141-000 Switch Matrix/COLUMN 8 -> unconnected-(U5-GPIO7-Pad9)
Routing:
- net /140-000 Keybaord/141-000 Switch Matrix/COLUMN 14: track 20.0 -> 240.8 mm
- net /140-000 Keybaord/141-000 Switch Matrix/COLUMN 13: track 21.9 -> 205.7 mm
- net /140-000 Keybaord/141-000 Switch Matrix/COLUMN 12: track 42.7 -> 187.3 mm
- net /140-000 Keybaord/141-000 Switch Matrix/ROW 1: track 229.4 -> 348.6 mm, vias 0 -> 2
- net /140-000 Keybaord/141-000 Switch Matrix/COLUMN 1: track 83.5 -> 197.7 mm
- net /140-000 Keybaord/141-000 Switch Matrix/COLUMN 11: track 65.7 -> 161.9 mm
- net /140-000 Keybaord/141-000 Switch Matrix/COLUMN 2: track 92.5 -> 183.1 mm
- net /140-000 Keybaord/141-000 Switch Matrix/COLUMN 10: track 65.7 -> 138.5 mm
- net /140-000 Keybaord/141-000 Switch Matrix/ROW 2: track 257.1 -> 328.2 mm, vias 0 -> 2
- net /140-000 Keybaord/141-000 Switch Matrix/COLUMN 3: track 89.7 -> 156.5 mm
- net /140-000 Keybaord/141-000 Switch Matrix/COLUMN 6: track 144.9 -> 93.7 mm, vias 0 -> 1
- net /140-000 Keybaord/141-000 Switch Matrix/ROW 3: track 248.1 -> 299.0 mm, vias 0 -> 2
- net /140-000 Keybaord/141-000 Switch Matrix/COLUMN 9: track 65.7 -> 115.2 mm, vias 0 -> 1
- net /140-000 Keybaord/141-000 Switch Matrix/COLUMN 7: track 65.7 -> 104.4 mm, vias 0 -> 1
- net /140-000 Keybaord/141-000 Switch Matrix/COLUMN 5: track 131.4 -> 95.6 mm
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- added copper zone on B.Cu, net +1V1
- added copper zone on B.Cu, net +3.3V
- added copper zone on B.Cu, net GND
- added copper zone on F.Cu, net GND
